File: pcb-covox-amp-v2.kicad_pcb (KiCad board)
At the start: 2 copper layers, 78 x 56 mm, 45 parts, among them J1 DB25, P1 USB, U1 LM386, X1 Amp, X2 Raw

Commit message: another commit
Parts:
- added C13: 4.7uF, Capacitors_SMD:C_0805_HandSoldering, F.Cu at (161.0, 134.5)
- added C14: 100nF, Capacitors_SMD:C_0805_HandSoldering, F.Cu at (157.5, 134.5)
- added C15: 100nF, Capacitors_SMD:C_0805_HandSoldering, F.Cu at (178.0, 119.0)
- added C16: 10nF, Capacitors_SMD:C_0805_HandSoldering, F.Cu at (182.5, 131.0)
- added FB1: FERRITE, Resistors_SMD:R_0805_HandSoldering, F.Cu at (179.5, 131.0)
- added P2: CONN_01X10, Pin_Headers:Pin_Header_Straight_1x10, F.Cu at (133.0, 101.4)
- added R21: 100, Resistors_SMD:R_0805_HandSoldering, F.Cu at (138.1, 101.4)
- added R22: 100, Resistors_SMD:R_0805_HandSoldering, F.Cu at (138.1, 103.9)
- added R23: 100, Resistors_SMD:R_0805_HandSoldering, F.Cu at (138.1, 106.4)
- added R24: 100, Resistors_SMD:R_0805_HandSoldering, F.Cu at (138.1, 109.0)
- added R25: 100, Resistors_SMD:R_0805_HandSoldering, F.Cu at (138.1, 111.5)
- added R26: 100, Resistors_SMD:R_0805_HandSoldering, F.Cu at (138.1, 114.1)
- added R27: 100, Resistors_SMD:R_0805_HandSoldering, F.Cu at (138.1, 116.6)
- added R28: 100, Resistors_SMD:R_0805_HandSoldering, F.Cu at (138.1, 119.1)
- added R29: 10K, Resistors_SMD:R_0805_HandSoldering, F.Cu at (176.5, 131.0)
- added U2: FT245RL, Housings_SSOP:SSOP-28_5.3x10.2mm_Pitch0.65mm, F.Cu at (169.5, 121.5)
- C12: value 0.1uF -> 100nF
- moved C5 22.7 mm to (162.5, 101.0), turned to 180 degrees
- moved C4 21.1 mm to (155.5, 115.5), turned to 90 degrees
- moved C12 20.2 mm to (187.0, 133.0)
- moved C1 19.6 mm to (146.5, 107.5), turned to 270 degrees
- moved U1 15.2 mm to (152.5, 108.0)
- moved R1 15.0 mm to (159.0, 105.5), turned to 180 degrees
- moved C3 13.8 mm to (160.0, 115.5), turned to 90 degrees
- moved C7 13.3 mm to (168.0, 109.5), turned to 180 degrees
- moved X2 12.1 mm to (184.0, 99.5)
- moved X1 11.5 mm to (183.9, 112.4)
- moved C6 11.1 mm to (151.0, 119.0)
- moved P1 10.3 mm to (187.4, 126.7)
- moved MH1 10.0 mm to (186.5, 89.5)
- moved MH2 10.0 mm to (186.5, 138.5)
- moved D1 9.51 mm to (181.0, 138.5)
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Connections:
- P1 pad 1: +5V -> Net-(C16-Pad1)
- P1 pad 2: (no net) -> USB_D-
- P1 pad 3: (no net) -> USB_D+
Routing:
- net +5V: track 46.4 -> 125.4 mm, vias 0 -> 2
- net Net-(R21-Pad2): track 0.00 -> 51.9 mm, vias 0 -> 2
- net Net-(R24-Pad2): track 0.00 -> 40.9 mm, vias 0 -> 2
- net Net-(R22-Pad2): track 0.00 -> 39.6 mm, vias 0 -> 2
- net Net-(R26-Pad2): track 0.00 -> 37.5 mm, vias 0 -> 2
- net Net-(R27-Pad2): track 0.00 -> 37.1 mm, vias 0 -> 2
- net Net-(R23-Pad2): track 0.00 -> 37.0 mm, vias 0 -> 2
- net Net-(R28-Pad2): track 0.00 -> 33.1 mm, vias 0 -> 2
- net Net-(R25-Pad2): track 0.00 -> 32.7 mm, vias 0 -> 2
- net GND: track 3.38 -> 34.8 mm, vias 0 -> 1
- net Input+: track 58.7 -> 29.0 mm
- net Data1: track 4.92 -> 28.1 mm
- net Data3: track 7.43 -> 30.5 mm
- net Data2: track 7.22 -> 30.2 mm
- net Data5: track 13.3 -> 36.1 mm
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Other:
- board size 78 x 56 mm -> 87 x 56 mm
- net class Default: trace_width 1 -> 0.4
- net class Micro-USB removed
- board text added: "Covox Amplifier v2 Rev 1 (July 2016) Designer: Yeo Kheng Meng"
- board text removed: "Covox Amplifier Rev 3 (July 2016) Designer: Yeo Kheng Meng"

Commit message: silkscreen
Parts:
- C3, C4, C6, C9: value 0.1uF -> 100nF
Other:
- board text added: "+5V"
- board text added: "D0"
- board text added: "D1"
- board text added: "D2"
- board text added: "D3"
- board text added: "D4"
- board text added: "D5"
- board text added: "D6"
- board text added: "D7"
- board text added: "GND"
