File: pcb-covox-amp-v2.sch (KiCad schematic (older format))
At the start: 45 parts, among them J1 DB25, P1 USB, U1 LM386, X1 Amp, X2 Raw

Commit message: another commit
Parts:
- added C13: 4.7uF, Capacitors_SMD:C_0805_HandSoldering, symbol C
- added C14, C15: 100nF, Capacitors_SMD:C_0805_HandSoldering, symbol C
- added C16: 10nF, Capacitors_SMD:C_0805_HandSoldering, symbol C
- added FB1: FERRITE, Resistors_SMD:R_0805_HandSoldering, symbol FERRITE
- added P2: CONN_01X10, Pin_Headers:Pin_Header_Straight_1x10, symbol CONN_01X10
- added R21, R22, R23, R24, R25, R26, R27, R28: 100, Resistors_SMD:R_0805_HandSoldering, symbol R
- added R29: 10K, Resistors_SMD:R_0805_HandSoldering, symbol R
- added U2: FT245RL, Housings_SSOP:SSOP-28_5.3x10.2mm_Pitch0.65mm, symbol FT245RL
- C12: value 0.1uF -> 100nF
Connections:
- net +5V: now also C13.1, C14.1, FB1.2, P2.10 (P10), R29.1, U2.20 (VCC), U2.4 (VCCIO); no longer P1.1 (VCC)
- net Data0: now also P2.1 (P1), R21.1
- net Data1: now also P2.2 (P2), R22.1
- net Data2: now also P2.3 (P3), R23.1
- net Data3: now also P2.4 (P4), R24.1
- net Data4: now also P2.5 (P5), R25.1
- net Data5: now also P2.6 (P6), R26.1
- net Data6: now also P2.7 (P7), R27.1
- net Data7: now also P2.8 (P8), R28.1
- net GND: now also C13.2, C14.2, C15.2, C16.2, P2.9 (P9), U2.18 (GND), U2.21 (GND), U2.25 (AGND), U2.26 (TEST), U2.7 (GND)
- net USB_D-: now reaches P1.2 (D-)
- net USB_D-: now also U2.16 (USBD-)
- net USB_D+: now reaches P1.3 (D+)
- net USB_D+: now also U2.15 (USBD+)
- new net: C16.1, FB1.1, P1.1 (VCC)
- new net: R21.2, U2.1 (D0)
- new net: R27.2, U2.10 (D6)
- new net: R24.2, U2.11 (D3)
- new net: R29.2, U2.12 (~PWREN)
- new net: C15.1, U2.17 (3V3OUT)
- new net: R25.2, U2.2 (D4)
- new net: R23.2, U2.3 (D2)
- new net: R22.2, U2.5 (D1)
- new net: R28.2, U2.6 (D7)
- new net: R26.2, U2.9 (D5)
Other:
- moved on the sheet: C1, C10, C11, C2, C3, C4, C5, C6, C7, D1, R1, R2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

Commit message: silkscreen
Parts:
- C3, C4, C6, C9: value 0.1uF -> 100nF
Changed lines of the file:
@@
 Sheet 1 1
 Title "Covox with Amplifier v2"
-Date "2016-07-24"
+Date "2016-07-25"
 Rev "1"
 Comp ""
@@
 P 5950 2550
 F 0 "C9" H 5975 2650 50  0000 L CNN
-F 1 "0.1uF" H 5975 2450 50  0000 L CNN
+F 1 "100nF" H 5975 2450 50  0000 L CNN
 F 2 "Capacitors_SMD:C_0805_HandSoldering" H 5988 2400 50  0001 C CNN
 F 3 "" H 5950 2550 50  0000 C CNN
@@
 P 2050 5850
 F 0 "C4" V 2100 5700 50  0000 L CNN
-F 1 "0.1uF" V 2000 5600 50  0000 L CNN
+F 1 "100nF" V 2000 5550 50  0000 L CNN
 F 2 "Capacitors_SMD:C_0805_HandSoldering" H 2088 5700 50  0001 C CNN
 F 3 "" H 2050 5850 50  0000 C CNN
@@
 P 2050 5450
 F 0 "C3" V 2100 5300 50  0000 L CNN
-F 1 "0.1uF" V 2000 5200 50  0000 L CNN
+F 1 "100nF" V 2000 5150 50  0000 L CNN
 F 2 "Capacitors_SMD:C_0805_HandSoldering" H 2088 5300 50  0001 C CNN
 F 3 "" H 2050 5450 50  0000 C CNN
@@
 P 3550 6700
 F 0 "C6" H 3650 6600 50  0000 L CNN
-F 1 "0.1uF" H 3300 6600 50  0000 L CNN
+F 1 "100nF" H 3300 6600 50  0000 L CNN
 F 2 "Capacitors_SMD:C_0805_HandSoldering" H 3588 6550 50  0001 C CNN
 F 3 "" H 3550 6700 50  0000 C CNN
